File: pcb/beartag.kicad_pcb (KiCad board)
At the start: 2 copper layers, 25.6 x 31 mm, 25 parts, among them J1 USB_C_Receptacle_USB2.0_14P, Q1 AO3401A, SW1 SW_Push, SW2 SW_Push, U1 CH571F, U2 XC6206P332MR, Y1 32 MHz, Y2 32.768 kHz

Commit message: pcb updates
Parts:
- added QR*****: qrcode, lcsc:qrcode, B.Cu at (29.3, 48.0)
- moved C2 3.77 mm to (25.4, 43.1), turned to 45 degrees
- moved AE1 2.52 mm to (24.6, 39.6)
- moved Y1 0.30 mm to (35.5, 44.4)
- moved Y2 0.11 mm to (26.4, 45.4)
Connections:
- U1 pad 17: unconnected-(U1-PB22/TMR3/RXD2-Pad17) -> BTN1
- U1 pad 25: BTN1 -> unconnected-(U1-PA15/MIS0/RXD0/AIN5-Pad25)
Routing:
- net GND: track 38.6 -> 18.8 mm, vias 16 -> 112
- net VICIA: track 11.5 -> 16.9 mm
- net BTN1: track 14.7 -> 18.3 mm, vias 0 -> 2
- net LED: track 9.94 -> 9.07 mm
- net X32MO: track 2.49 -> 3.26 mm
- net +5V: track 21.4 -> 20.6 mm
- net X32MI: track 7.11 -> 7.71 mm
- net ANT: track 11.7 -> 11.1 mm
- added copper zone on F.Cu, net +5V
- added copper zone on F.Cu, net ANT
- added copper zone on F.Cu, net D+
- added copper zone on F.Cu, net D-
- added copper zone on F.Cu, net GND
Other:
- board size 25.6 x 31 mm -> 25.6 x 33.7 mm
- board text added: "70274a6"
- board text added: "BTN 1"
- board text added: "RST"
- board text added: "v2"
- board text removed: "COMMIT"
- board text removed: "v1"
